File: VCO/VCO.kicad_pcb (KiCad board)
At the start: 2 copper layers, 46 parts, among them J1 Conn_01x05, Q1 MMBFJ112, T1 220k, T2 25k, T3 10k, U3 OPA2134, U5 LM311, U6 TL074, U7 TL074

Commit message: Schematic is almost complete
Parts:
- added C12: 47p, Capacitor_THT:C_Disc_D4.7mm_W2.5mm_P5.00mm, F.Cu at (125.7, 168.9)
- added D3: 1N4148, Diode_THT:D_DO-35_SOD27_P7.62mm_Horizontal, F.Cu at (319.4, 107.2)
- added D4: 1N4148, Diode_THT:D_DO-35_SOD27_P7.62mm_Horizontal, F.Cu at (332.7, 99.1)
- added D5: 1N4148, Diode_THT:D_DO-35_SOD27_P7.62mm_Horizontal, F.Cu at (359.4, 162.6)
- added D6: 1N4148, Diode_THT:D_DO-35_SOD27_P7.62mm_Horizontal, F.Cu at (359.4, 166.1)
- added J2: WAVE_OUT, Connector_PinSocket_2.54mm:PinSocket_1x05_P2.54mm_Vertical, F.Cu at (108.0, 179.1)
- added R27: 100k, Resistor_THT:R_Axial_DIN0207_L6.3mm_D2.5mm_P10.16mm_Horizontal, F.Cu at (361.9, 125.7)
- added R28: 10k, Resistor_THT:R_Axial_DIN0207_L6.3mm_D2.5mm_P10.16mm_Horizontal, F.Cu at (361.9, 129.8)
- added R29: 100k 1%, Resistor_THT:R_Axial_DIN0207_L6.3mm_D2.5mm_P10.16mm_Horizontal, F.Cu at (319.4, 91.2)
- added R30: 100k 1%, Resistor_THT:R_Axial_DIN0207_L6.3mm_D2.5mm_P10.16mm_Horizontal, F.Cu at (319.4, 95.3)
- added R31: 100k 1%, Resistor_THT:R_Axial_DIN0207_L6.3mm_D2.5mm_P10.16mm_Horizontal, F.Cu at (332.7, 91.2)
- added R32: 50k 1%, Resistor_THT:R_Axial_DIN0207_L6.3mm_D2.5mm_P10.16mm_Horizontal, F.Cu at (319.4, 99.3)
- added R33: 100k, Resistor_THT:R_Axial_DIN0207_L6.3mm_D2.5mm_P10.16mm_Horizontal, F.Cu at (77.5, 162.6)
- added R37: 10k, Resistor_THT:R_Axial_DIN0207_L6.3mm_D2.5mm_P10.16mm_Horizontal, F.Cu at (361.9, 133.8)
- added R38: 4k7, Resistor_THT:R_Axial_DIN0207_L6.3mm_D2.5mm_P10.16mm_Horizontal, F.Cu at (99.1, 171.4)
- added R39: 1k, Resistor_THT:R_Axial_DIN0207_L6.3mm_D2.5mm_P10.16mm_Horizontal, F.Cu at (88.9, 176.5)
- added R40: 1k, Resistor_THT:R_Axial_DIN0207_L6.3mm_D2.5mm_P10.16mm_Horizontal, F.Cu at (83.8, 153.7)
- added R41: 200k 1%, Resistor_THT:R_Axial_DIN0207_L6.3mm_D2.5mm_P10.16mm_Horizontal, F.Cu at (120.7, 174.0)
- added R42: 1k, Resistor_THT:R_Axial_DIN0207_L6.3mm_D2.5mm_P10.16mm_Horizontal, F.Cu at (114.3, 163.8)
- added R43: 150k, Resistor_THT:R_Axial_DIN0207_L6.3mm_D2.5mm_P10.16mm_Horizontal, F.Cu at (346.1, 158.8)
- added R44: 150k, Resistor_THT:R_Axial_DIN0207_L6.3mm_D2.5mm_P10.16mm_Horizontal, F.Cu at (142.2, 171.4)
- added R45: 1k5, Resistor_THT:R_Axial_DIN0207_L6.3mm_D2.5mm_P10.16mm_Horizontal, F.Cu at (346.1, 162.8)
- added R46: 15k, Resistor_THT:R_Axial_DIN0207_L6.3mm_D2.5mm_P10.16mm_Horizontal, F.Cu at (346.1, 166.9)
- added R47: 1k, Resistor_THT:R_Axial_DIN0207_L6.3mm_D2.5mm_P10.16mm_Horizontal, F.Cu at (142.2, 176.5)
- added R48: 22k, Resistor_THT:R_Axial_DIN0207_L6.3mm_D2.5mm_P10.16mm_Horizontal, F.Cu at (346.1, 170.9)
- added R52: 470k, Resistor_THT:R_Axial_DIN0207_L6.3mm_D2.5mm_P10.16mm_Horizontal, F.Cu at (375.3, 137.9)
- added T4: 47k, Connector_PinHeader_2.54mm:PinHeader_1x03_P2.54mm_Vertical, F.Cu at (346.8, 91.5)
- moved R11 184.4 mm to (308.7, 41.4)
- moved R15 184.4 mm to (322.0, 57.6)
- moved R16 184.4 mm to (295.4, 33.3)
- moved R23 184.4 mm to (322.0, 53.6)
- moved R24 184.4 mm to (308.7, 53.6)
- moved R3 184.4 mm to (295.4, 37.4)
- moved R4 184.4 mm to (308.7, 33.3)
- moved R5 184.4 mm to (295.4, 41.4)
- moved R50 184.4 mm to (322.0, 61.7)
- moved R51 184.4 mm to (308.7, 49.5)
- moved R6 184.4 mm to (308.7, 37.4)
- moved R8 184.4 mm to (295.4, 49.5)
- moved R9 184.4 mm to (322.0, 33.3)
- moved C8 184.4 mm to (365.8, 47.0)
- moved D2 184.4 mm to (335.3, 56.9)
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Connections:
- U6 pad 10: (no net) -> Net-(R52-Pad2)
- U6 pad 12: (no net) -> GND
- U6 pad 13: (no net) -> Net-(R27-Pad2)
- U6 pad 14: (no net) -> Net-(R33-Pad2)
- U6 pad 8: (no net) -> Net-(R37-Pad1)
- U6 pad 9: (no net) -> Net-(R28-Pad2)
- U7 pad 10: (no net) -> GND
- U7 pad 12: (no net) -> Net-(D5-Pad2)
- U7 pad 13: (no net) -> Net-(R45-Pad2)
- U7 pad 14: (no net) -> Net-(R46-Pad2)
- U7 pad 5: (no net) -> GND
- U7 pad 6: (no net) -> Net-(D3-Pad1)
- U7 pad 7: (no net) -> Net-(D3-Pad2)
- U7 pad 8: (no net) -> Net-(C12-Pad1)
- U7 pad 9: (no net) -> Net-(C12-Pad2)

Commit message: Introduced a PCB
Parts:
- added C5: 100n, Capacitor_THT:C_Rect_L7.0mm_W2.0mm_P5.00mm, F.Cu at (153.7, 44.5)
- moved R49 167.4 mm to (176.5, 86.4), turned to 180 degrees
- moved R4 145.0 mm to (170.2, 76.2)
- moved R6 141.9 mm to (170.2, 68.6)
- moved R50 141.7 mm to (180.3, 55.9)
- moved R16 137.9 mm to (157.5, 31.8)
- moved R3 132.2 mm to (170.2, 80.0)
- moved R5 128.9 mm to (170.2, 72.4)
- moved R8 119.3 mm to (176.5, 59.7)
- moved R7 116.6 mm to (180.3, 64.8), turned to 180 degrees
- moved T1 52.2 mm to (186.7, 44.5)
- moved T2 49.9 mm to (152.0, -7.62)
- moved R10 26.7 mm to (139.7, 25.4)
- moved U3 24.1 mm to (142.2, 52.1)
- moved C7 22.9 mm to (147.3, 35.6)
- moved R14 20.3 mm to (149.9, 25.4)
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Connections:
- U3 pad 4: (no net) -> VSS
- U3 pad 8: (no net) -> VDD

Commit message: Updated .gitignore and added more footprints
Parts:
- removed the C8 at (365.8, 47.0)
- C8: footprint Capacitor_THT:C_Disc_D4.7mm_W2.5mm_P5.00mm -> Capacitor_THT:C_Axial_L5.1mm_D3.1mm_P10.00mm_Horizontal
- J1: footprint Connector_PinSocket_1.27mm:PinSocket_1x05_P1.27mm_Vertical -> Connector_PinSocket_2.54mm:PinSocket_1x05_P2.54mm_Vertical
- T1, T2, T3, T4: footprint Connector_PinHeader_2.54mm:PinHeader_1x03_P2.54mm_Vertical -> Potentiometer_THT:Potentiometer_Bourns_3266Y_Vertical
- U3, U5: footprint Package_DIP:DIP-8_W10.16mm -> Package_DIP:DIP-8_W7.62mm
- moved T4 176.0 mm to (170.8, 92.1)
- moved J1 165.5 mm to (185.4, 55.9)
- moved C8 115.0 mm to (104.8, 52.1)
- moved U6 83.5 mm to (139.1, 71.8)
- moved Q1 68.0 mm to (104.8, 47.6)
- moved R22 64.3 mm to (118.7, 27.3)
- moved T2 63.8 mm to (145.4, 55.9), turned to 270 degrees
- moved U7 62.6 mm to (161.3, 73.7)
- moved R13 58.3 mm to (121.9, 33.0)
- moved C11 57.6 mm to (129.5, 29.8)
- moved R33 57.4 mm to (101.6, 110.5)
- moved R39 57.4 mm to (113.0, 124.5)
- moved R41 57.4 mm to (144.8, 121.9)
- moved R42 57.4 mm to (138.4, 111.8)
- moved R47 57.4 mm to (166.4, 124.5)
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Other:
- board outline added: 100.3 x 72.4 mm

Commit message: Almost finished the schematic
Parts:
- added C1: 22u, Capacitor_THT:CP_Radial_D8.0mm_P3.80mm, F.Cu at (196.8, 38.1)
- added C13: 100n, Capacitor_THT:C_Rect_L7.0mm_W2.0mm_P5.00mm, F.Cu at (160.7, 75.6)
- added C2: 22u, Capacitor_THT:CP_Radial_D8.0mm_P3.80mm, F.Cu at (200.0, 91.4)
- added C3: 100n, Capacitor_THT:C_Rect_L7.0mm_W2.0mm_P5.00mm, F.Cu at (185.4, 43.8)
- added C4: 100n, Capacitor_THT:C_Rect_L7.0mm_W2.0mm_P5.00mm, F.Cu at (192.4, 64.1)
- added C6: 100n, Capacitor_THT:C_Rect_L7.0mm_W2.0mm_P5.00mm, F.Cu at (120.7, 73.0)
- added J3: POWER_SUPPLY_+15_-15, Connector_PinSocket_2.54mm:PinSocket_1x02_P2.54mm_Vertical, F.Cu at (186.1, 76.2)
- added J4: YUSYNTH_PWM, Connector_PinSocket_2.54mm:PinSocket_1x04_P2.54mm_Vertical, F.Cu at (261.5, -3.25)
- added R1: 10, Resistor_THT:R_Axial_DIN0207_L6.3mm_D2.5mm_P10.16mm_Horizontal, F.Cu at (193.0, 38.1)
- added R2: 10, Resistor_THT:R_Axial_DIN0207_L6.3mm_D2.5mm_P10.16mm_Horizontal, F.Cu at (193.0, 86.4)
- added R34: 180k, Resistor_THT:R_Axial_DIN0207_L6.3mm_D2.5mm_P10.16mm_Horizontal, F.Cu at (247.5, -3.55)
- added R35: 100k, Resistor_THT:R_Axial_DIN0207_L6.3mm_D2.5mm_P10.16mm_Horizontal, F.Cu at (247.5, 0.50)
- added U1: L78L15_TO92, Package_TO_SOT_THT:TO-92_Inline, F.Cu at (188.6, 48.3)
- added U2: L78L15_TO92, Package_TO_SOT_THT:TO-92_Inline, F.Cu at (196.8, 69.8)
- moved R46 201.2 mm to (162.6, 84.5)
- moved D5 198.1 mm to (176.5, 86.4)
- moved D6 191.3 mm to (184.2, 89.5), turned to 180 degrees
- moved R43 173.7 mm to (179.1, 111.1)
- moved R45 173.7 mm to (179.1, 115.2)
- moved R48 173.7 mm to (179.1, 123.3)
- moved R12 16.9 mm to (82.5, 88.3)
- moved R3 5.72 mm to (167.0, 66.0)
- moved R4 5.72 mm to (167.0, 63.5)
- moved R49 5.72 mm to (173.4, 70.5)
- moved R5 5.72 mm to (167.0, 61.0)
- moved R50 5.72 mm to (174.6, 49.5)
- moved R6 5.72 mm to (167.0, 58.4)
- moved R7 5.72 mm to (177.2, 55.9)
- moved R8 5.72 mm to (172.1, 52.7)
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Connections:
- net /5 renamed Net-(J1-Pad5)
- net /6 renamed Net-(C9-Pad1)
- net /7 renamed Net-(J1-Pad4)
- net /8 renamed Net-(J1-Pad3)
- net /9 renamed Net-(J1-Pad2)
- C9 pad 2: /2 -> Net-(C9-Pad2)
- J1 pad 1: /1 -> Net-(J1-Pad1)
- J2 pad 2: /1 -> Net-(J2-Pad2)
- R16 pad 2: /2 -> Net-(R16-Pad2)
- R17 pad 2: /2 -> Net-(C9-Pad2)
- R36 pad 1: /3 -> Net-(J4-Pad2)
- R47 pad 2: /1 -> Net-(J2-Pad2)
- R51 pad 1: /4 -> Net-(J4-Pad4)
- R7 pad 1: /1 -> Net-(J1-Pad1)
- U6 pad 11: (no net) -> VSS
- U6 pad 4: (no net) -> VDD
- U7 pad 11: (no net) -> VSS
- U7 pad 4: (no net) -> VDD

Commit message: Updated LM394 footprint and placed some elements on the PCB
Parts:
- removed J2: WAVE_OUT, Connector_PinSocket_2.54mm:PinSocket_1x05_P2.54mm_Vertical
- added CON2: Linear FM, Connector_PinSocket_2.54mm:PinSocket_1x05_P2.54mm_Vertical, F.Cu at (172.7, -8.26)
- added CON3: Sync in, Connector_PinSocket_2.54mm:PinSocket_1x05_P2.54mm_Vertical, F.Cu at (177.3, -8.26)
- added CON5: Wave output, Connector_PinSocket_2.54mm:PinSocket_1x05_P2.54mm_Vertical, F.Cu at (148.0, 95.2)
- added U4: LM394CN, Package_DIP:DIP-8_W7.62mm, F.Cu at (119.4, 43.8)
- CON1: renamed from J1; value Conn_01x05 -> Modulation
- CON4: renamed from J4; value YUSYNTH_PWM -> PWM input
- CON6: renamed from J3; value POWER_SUPPLY_+15_-15 -> Input +/- 15V
- R12: value 1k TEMPCO -> 1k NTC tempco
- U1: value L78L15_TO92 -> L78L15
- U2: value L78L15_TO92 -> L79L15
- U3: value OPA2134 -> OPA2137
- moved R52 280.2 mm to (106.0, 60.3)
- moved R37 245.7 mm to (120.7, 87.6)
- moved R25 227.7 mm to (108.0, 54.6)
- moved R36 222.7 mm to (114.3, 76.8), turned to 90 degrees
- moved D2 203.9 mm to (131.4, 52.1), turned to 180 degrees
- moved R26 200.3 mm to (135.9, 64.1)
- moved R51 198.9 mm to (110.5, 66.7), turned to 270 degrees
- moved R15 190.4 mm to (133.3, 31.8), turned to 270 degrees
- moved R23 188.9 mm to (133.3, 64.1), turned to 180 degrees
- moved R24 182.9 mm to (125.7, 55.2)
- moved R30 173.4 mm to (149.9, 59.1)
- moved R53 172.5 mm to (136.5, 33.7), turned to 270 degrees
- moved R21 172.2 mm to (149.9, 52.1), turned to 180 degrees
- moved CON4 167.8 mm to (118.1, 83.8), turned to 270 degrees
- moved R11 167.2 mm to (141.6, 48.9), turned to 180 degrees
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Connections:
- net Net-(C9-Pad2) renamed /HARD_SYNC_IN
- net Net-(J1-Pad1) renamed /COARSE_TUNE
- net Net-(J1-Pad2) renamed /FINE_TUNE
- net Net-(J1-Pad5) renamed /EXP_FM
- net Net-(J4-Pad1) renamed /PWM_IN
- net Net-(J4-Pad3) renamed /PW_POT
- C9 pad 1: Net-(C9-Pad1) -> /SOFT_SYNC_IN
- CON1 pad 3: Net-(J1-Pad3) -> /V\OCT_IN
- CON1 pad 4: Net-(J1-Pad4) -> /V\OCT_IN
- CON4 pad 2: Net-(J4-Pad2) -> +15V
- CON4 pad 4: Net-(J4-Pad4) -> -15V
- CON6 pad 1: Net-(J3-Pad1) -> +15V
- CON6 pad 2: Net-(J3-Pad2) -> GND
- R1 pad 2: Net-(J3-Pad1) -> +15V
- R16 pad 2: Net-(R16-Pad2) -> /LINEAR_FM
- R2 pad 2: Net-(J3-Pad2) -> -15V
- R36 pad 1: Net-(J4-Pad2) -> +15V
- R39 pad 2: Net-(J2-Pad3) -> /TRI_OUT
- R4 pad 2: Net-(J1-Pad4) -> /V\OCT_IN
- R40 pad 2: Net-(J2-Pad5) -> /PULSE_OUT
- R42 pad 2: Net-(J2-Pad4) -> /SAW_OUT
- R47 pad 2: Net-(J2-Pad2) -> /SINE_OUT
- R5 pad 2: Net-(J1-Pad3) -> /V\OCT_IN
- R51 pad 1: Net-(J4-Pad4) -> -15V
- R9 pad 1: Net-(R9-Pad1) -> Net-(R3-Pad1)
- U1 pad 3: Net-(J3-Pad1) -> +15V
- U2 pad 1: Net-(J3-Pad2) -> -15V
- U3 pad 2: Net-(R9-Pad1) -> Net-(R3-Pad1)
Routing:
- net Net-(C11-Pad2): track 0.00 -> 22.9 mm
- net Net-(C8-Pad2): track 0.00 -> 15.9 mm
- net Net-(C8-Pad1): track 0.00 -> 4.45 mm
- net GND: track 0.00 -> 3.70 mm
- net Net-(C10-Pad2): track 0.00 -> 3.07 mm

Commit message: Updated PCB
Parts:
- removed CON2: Linear FM, Connector_PinSocket_2.54mm:PinSocket_1x05_P2.54mm_Vertical
- CON3: value Sync in -> Sync_In; footprint Connector_PinSocket_2.54mm:PinSocket_1x05_P2.54mm_Vertical -> Connector_PinSocket_2.54mm:PinSocket_1x04_P2.54mm_Vertical
- CON6: footprint Connector_PinSocket_2.54mm:PinSocket_1x02_P2.54mm_Vertical -> Connector_PinSocket_2.54mm:PinSocket_1x03_P2.54mm_Vertical
- moved CON3 42.0 mm to (191.6, 31.2)
- moved T1 26.7 mm to (185.7, 66.0), turned to 270 degrees
- moved R16 23.6 mm to (175.3, 37.7)
- moved CON6 19.8 mm to (198.8, 61.0)
- moved C10 18.8 mm to (179.6, 49.5)
- moved R53 18.6 mm to (142.4, 51.3), turned to 90 degrees
- moved R21 18.6 mm to (156.7, 69.3)
- moved T2 17.4 mm to (154.9, 54.2), turned to 90 degrees
- moved R50 16.4 mm to (189.2, 53.6), turned to 180 degrees
- moved U5 16.4 mm to (183.4, 50.8)
- moved R18 15.9 mm to (170.2, 42.2)
- moved R17 15.8 mm to (173.2, 52.3)
- moved R15 15.4 mm to (145.5, 41.1)
- moved C9 15.3 mm to (188.2, 37.8), turned to 90 degrees
- moved C3 13.7 mm to (189.2, 56.5), turned to 270 degrees
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Connections:
- C13 pad 1: VDD -> +15V
- C13 pad 2: VSS -> -15V
- C3 pad 1: VDD -> VCC
- C5 pad 1: VDD -> VCC
- C6 pad 1: VDD -> +15V
- C6 pad 2: VSS -> -15V
- CON1 pad 3: /V\OCT_IN -> /V\OCT_IN2
- CON1 pad 4: /V\OCT_IN -> /V\OCT_IN1
- CON3 pad 1: /HARD_SYNC_IN -> GND
- CON3 pad 2: /SOFT_SYNC_IN -> /HARD_SYNC_IN
- CON3 pad 3: (no net) -> /SOFT_SYNC_IN
- CON3 pad 4: (no net) -> /FMMOD
- CON6 pad 1: +15V -> /+15VPS
- R1 pad 2: +15V -> /+15VPS
- R16 pad 2: /LINEAR_FM -> /FMMOD
- R2 pad 2: -15V -> /-15VPS
- R4 pad 2: /V\OCT_IN -> /V\OCT_IN1
- R5 pad 2: /V\OCT_IN -> /V\OCT_IN2
- U1 pad 1: VDD -> VCC
- U1 pad 3: +15V -> /+15VPS
- U2 pad 1: -15V -> /-15VPS
- U3 pad 8: VDD -> VCC
- U5 pad 1: GND -> VSS
- U5 pad 4: GND -> VSS
- U6 pad 11: VSS -> -15V
- U6 pad 4: VDD -> +15V
- U7 pad 11: VSS -> -15V
- U7 pad 4: VDD -> +15V
Routing:
- net VCC: track 0.00 -> 45.4 mm
- net Net-(R3-Pad1): track 0.00 -> 37.0 mm
- net +15V: track 0.00 -> 25.2 mm
- net Net-(C7-Pad1): track 0.00 -> 23.1 mm
- net Net-(C11-Pad2): track 22.9 -> 0.00 mm
- net /HARD_SYNC_IN: track 0.00 -> 22.7 mm
- net GND: track 3.70 -> 24.1 mm
- net -15V: track 0.00 -> 18.7 mm
- net Net-(C10-Pad1): track 0.00 -> 17.4 mm
- net VSS: track 0.00 -> 16.6 mm
- net Net-(C8-Pad2): track 15.9 -> 0.00 mm
- net Net-(R10-Pad2): track 0.00 -> 12.9 mm
- net Net-(C10-Pad2): track 3.07 -> 13.5 mm
- net Net-(C7-Pad2): track 0.00 -> 10.1 mm
- net /+15VPS: track 0.00 -> 9.42 mm
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Other:
- net class Default: trace_width 0.25 -> 0.35
- rule trace_min: 0.2 -> 0.35
